File: CAN-Cape/CANcape.sch (EAGLE design)
At the start: 3 parts

Commit message: waiting on reformatting into mm of components
Connections:
- new net STANDBY: U$1.11
Changed lines of the file:
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@@
 <setting verticaltext="up"/>
 </settings>
-<grid distance="1" unitdist="mm" unit="mm" style="lines" multiple="1" display="no" altdistance="0.01" altunitdist="inch" altunit="inch"/>
+<grid distance="0.001" unitdist="mm" unit="mm" style="lines" multiple="1" display="no" altdistance="0.01" altunitdist="inch" altunit="inch"/>
 <layers>
 <layer number="1" name="Top" color="4" fill="1" visible="no" active="no"/>
@@
 </segment>
 </net>
+<net name="STANDBY" class="0">
+<segment>
+<pinref part="U$1" gate="G$1" pin="11"/>
+<wire x1="14" y1="71" x2="9" y2="71" width="0.1524" layer="91"/>
+</segment>
+</net>
